File: NVRTC.sch (KiCad schematic (older format))
At the start: 4 parts

Commit message: Rev 4
Parts:
- removed RTC1: ds1554p-70+, lib_fp:ds1554p-70+rev2, symbol RTC:ds1554p-70+
- added U1: M48T37Y, lib_fp:STM-SOH-44, symbol RTC:M48T37Y
Connections:
- net +5V: now also U1.38 (A13), U1.44 (Vcc), U1.5 (A14)
- net A0: now also U1.17 (A0)
- net A1: now also U1.16 (A1)
- net A10: now also U1.31 (A10)
- net A11: now also U1.35 (A11)
- net A12: now also U1.6 (A12)
- net A2: now also U1.15 (A2)
- net A3: now also U1.11 (A3)
- net A4: now also U1.10 (A4)
- net A5: now also U1.9 (A5)
- net A6: now also U1.8 (A6)
- net A7: now also U1.7 (A7)
- net A8: now also U1.37 (A8)
- net A9: now also U1.36 (A9)
- net ChipEnable: now also U1.30 (~E)
- net D0: now also U1.18 (DQ0)
- net D1: now also U1.19 (DQ1)
- net D2: now also U1.20 (DQ2)
- net D3: now also U1.24 (DQ3)
- net D4: now also U1.25 (DQ4)
- net D5: now also U1.26 (DQ5)
- net D6: now also U1.27 (DQ6)
- net D7: now also U1.28 (DQ7)
- net GND: now also U1.22 (Vss)
- net IRQ: now also U1.40 (~IRQ~/FT)
- net OutputEnable: now also U1.34 (~G)
- net RST: now also U1.2 (~RST~)
- net WriteEnable: now also U1.39 (~W)
- no-connect marks 0 -> 1
Other:
- note removed: "PIN ASSIGNMENT\nDS1554X -> M48T59\n=============\nPIN DS1554P\n=============\n1 26 \n2 NC \n3 NC \n4 1 \n5 28 \n6 27 \n7 22 \n8 20 \n9 19 \n10 18 \n11 17 \n12 16 \n13 15 \n14 13 \n15 12 \n16 11 \n17 14 \n18 10 \n19 9 \n20 8 \n21 7 \n22 6 \n23 5 \n24 4 \n25 3 \n26 25 \n27 24 \n28 21 \n29 23 \n30 2 \n31 28 \n32 28 \n33 NC \n34 NC"
- moved on the sheet: C1, C2, H1
